Commit message: ldlidar - add frame to the urdf, reference the node directly

File: mini_pupper_description/urdf/mini_pupper_description.urdf (robot description, URDF)
Before this commit: robot mini_pupper_description, 38 links, 37 joints
Links:
- added link lidar_frame, mass 0.001
Joints:
- added joint base_link_lidar_frame_joint: type fixed, parent base_link, child lidar_frame, origin xyz=0.0 -0.05 0.03 rpy=0 0 1.57

Commit message: URDF: Fix lidar position

File: mini_pupper_description/urdf/mini_pupper_description.urdf (robot description, URDF)
Before this commit: robot mini_pupper_description, 39 links, 38 joints
Joints:
- removed joint base_link_lidar_frame_joint
- added joint lidar_lidar_frame_joint: type fixed, parent lidar, child lidar_frame, origin xyz=0 0 0 rpy=0 0 1.57

Commit message: URDF: Fix lidar position

File: mini_pupper_description/urdf/mini_pupper_description.urdf (robot description, URDF)
Before this commit: robot mini_pupper_description, 29 links, 28 joints
Joints:
- joint lidar_joint: origin xyz=0.0 -0.05 0.03 rpy=0 0 1.57 -> xyz=0 0 0 rpy=0 0 1.57; parent base_link -> lidar
